File: Hardware/Schematic.sch (EAGLE design)
At the start: 105 parts, among them IC1 BQ25180YBGR, IC2 DRV2605YZFR, IC3 BMA421, IC9 RT6160AWSC, J1 503480-2400, J2 TC2030-IDC, J4 KH-TYPE-C-16P, Q1 20V/4.2A/52mΩ/1.4W, Q3 SI1308EDL-T1-GE3, U1 NRF52840_QF, U3 MAX17048G+T10, X1 32MHz, X2 32.768kHz

Commit message: Add files via upload
schematic final - modificare denumire label
Connections:
- net EPD_BUSY/1.5D renamed EPD_BUSY
- net EPS_BUSY/2.2D renamed EPS_BUSY
- removed net 3V3/1.7D: C34.2, IC2.VDD, Q1.S, R5.2, R7.2, R8.2, R_PWR_EPD.2
- removed net 3V3/2.4A: C12.1, C14.1, C19.1, C25.1, C33.1, C6.1, C7.1, C8.1, IC3.CSB, IC3.VDD, IC3.VDDIO, IC9.VOUT_1, IC9.VOUT_2, J2.1, R17.1, R18.1, TP_3.3V.TP, TP_3V3.TP, U1.VDD@A22, U1.VDD@AD14, U1.VDD@AD23, U1.VDD@B1, U1.VDD@W1, U1.VDDH@Y2
- removed net ALERT/1.6C: U3.!ALERT
- removed net ALERT/2.5C: U1.P0.10/NFC2@J24
- removed net D+/1.5D: D3.I/O2_2
- removed net D-/1.5D: D3.I/O1_2
- removed net D-/2.7D: U1.D+@AD6, U1.D-@AD4
- removed net EPD_CS.1.4C: J1.12
- removed net EPD_CS/2.2D: U1.P0.05/AIN3@K2
- removed net EPD_DC/1.5D: J1.11
- removed net EPD_DC/2.2D: U1.P0.15@AD10
- removed net EPD_RST/1.5D: J1.10
- removed net EPD_RST/2.2D: U1.P0.16@AC11
- removed net HAPTIC_EN/1.4C: IC2.EN
- removed net HAPTIC_EN/2.6A: U1.P0.12@U1
- removed net MOSI/1.5B: J1.14
- removed net MOSI/2.2D: U1.P0.03/AIN1@B13
- removed net P0.13/1.5D: C30.1, R5.1, SW_UP.2
- removed net P0.13/2.6C: U1.P0.13@AD8
- removed net P0.14/1.5D: C31.1, R8.1, SW_NET.2
- removed net P0.14/2.7C: U1.P0.14@AC9
- removed net P1.01/1.6C: Q1.G, R_PWR_EPD.1
- removed net P1.01/2.4B: U1.P1.01@Y23
- removed net P1.02/1.6C: C29.1, R7.1, SW_DN.2
- removed net P1.02/2.8C: U1.P1.02@W24
- removed net SCK/1.5B: J1.13
- removed net SCK/2.2D: U1.P0.02/AIN0@A12
- removed net SCL/1.4C: IC2.SCL, U3.SCL
- removed net SCL/2.4C: IC1.SCL, IC3.SCX, R17.2, R4.1, TP_SCL.TP, U1.P0.07@M2
- removed net SDA/1.4C: IC2.SDA, U3.SDA
- removed net SDA/2.4C: IC1.SDA, IC3.SDX, R18.2, R2.1, TP_SDA.TP, U1.P0.06@L1
- removed net VBAT/1.2A: C27.2, TP_VBAT.TP, U3.CELL, U3.VDD
- removed net VBAT/2.5C: C37.1, IC1.BAT
- removed net VBUS/1.5D: C42.1, C43.1, D3.VBUS, J4.VBUS
- removed net VBUS/2.6D: C21.1, C38.2, IC1.IN, U1.VBUS@AD2
- new net 3V3: C12.1, C14.1, C19.1, C25.1, C33.1, C34.2, C6.1, C7.1, C8.1, IC2.VDD, IC3.CSB, IC3.VDD, IC3.VDDIO, IC9.VOUT_1, IC9.VOUT_2, J2.1, Q1.S, R17.1, R18.1, R5.2, R7.2, R8.2, R_PWR_EPD.2, TP_3.3V.TP, TP_3V3.TP, U1.VDD@A22, U1.VDD@AD14, U1.VDD@AD23, U1.VDD@B1, U1.VDD@W1, U1.VDDH@Y2
- new net ALERT: U1.P0.10/NFC2@J24, U3.!ALERT
- new net D+: D3.I/O2_2, U1.D+@AD6
- new net D-: D3.I/O1_2, U1.D-@AD4
- new net EPD_CS: J1.12, U1.P0.05/AIN3@K2
- new net EPD_DC: J1.11, U1.P0.15@AD10
- new net EPD_RST: J1.10, U1.P0.16@AC11
- new net HAPTIC_EN: IC2.EN, U1.P0.12@U1
- new net MOSI: J1.14, U1.P0.03/AIN1@B13
- new net P0.13: C30.1, R5.1, SW_UP.2, U1.P0.13@AD8
- new net P0.14: C31.1, R8.1, SW_NET.2, U1.P0.14@AC9
- new net P1.01: Q1.G, R_PWR_EPD.1, U1.P1.01@Y23
- new net P1.02: C29.1, R7.1, SW_DN.2, U1.P1.02@W24
- new net SCK: J1.13, U1.P0.02/AIN0@A12
- new net SCL: IC1.SCL, IC2.SCL, IC3.SCX, R17.2, R4.1, TP_SCL.TP, U1.P0.07@M2, U3.SCL
- new net SDA: IC1.SDA, IC2.SDA, IC3.SDX, R18.2, R2.1, TP_SDA.TP, U1.P0.06@L1, U3.SDA
- new net VBAT: C27.2, C37.1, IC1.BAT, TP_VBAT.TP, U3.CELL, U3.VDD
- new net VBUS: C21.1, C38.2, C42.1, C43.1, D3.VBUS, IC1.IN, J4.VBUS, U1.VBUS@AD2

Commit message: varianta finala
Other:
- moved on the sheet: ANT1, C1, C1-EP-DR, C10, C11, C12, C13, C14, C15, C16, C17, C18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
